Commit message: Changed the ankle joint limits to accomodate for 2 degree incline

File: env-setup/humanoid.urdf (robot description, URDF)
Before this commit: robot dumpUrdf, 16 links, 15 joints
Joints:
- joint chest: type spherical -> fixed
- joint left_ankle: limit lower=-0.785 upper=0. effort=1000.0 velocity=0.5 -> lower=-0.785 upper=0.2094 effort=0.0 velocity=0.5; origin xyz=0.000000 -1.639480 0.000000 rpy=0 0 0 -> xyz=0.000000 -1.639480 0.000000 rpy=0 0 0.2094
- joint left_elbow: limit lower=0 upper=3.14 effort=1000.0 velocity=0.5 -> lower=0 upper=3.14 effort=0.0 velocity=0.5; type revolute -> fixed
- joint left_hip: limit lower=-1.57 upper=1.57 effort=1000.0 velocity=0.5 -> lower=-1.57 upper=1.57 effort=0.0 velocity=0.5; origin xyz=0.000000 0.000000 -0.339548 rpy=0 0 0 -> xyz=0.000000 0.000000 -0.339548 rpy=0 0 0.384
- joint left_knee: limit lower=-3.14 upper=0. effort=1000.0 velocity=0.5 -> lower=-3.14 upper=0. effort=0.0 velocity=0.5; origin xyz=0.000000 -1.686184 0.000000 rpy=0 0 0 -> xyz=0.000000 -1.686184 0.000000 rpy=0 0 -0.4712
- joint left_shoulder: type spherical -> fixed
- joint neck: type spherical -> fixed
- joint right_ankle: axis (none) -> 0.000000 0.000000 1.000000; limit (none) -> lower=-0.785 upper=0.2094 effort=0.0 velocity=0.5; origin xyz=0.000000 -1.639480 0.000000 rpy=0 0 0 -> xyz=0.000000 -1.639480 0.000000 rpy=0 0 0.2094; type fixed -> revolute
- joint right_elbow: limit lower=0 upper=3.14 effort=1000.0 velocity=0.5 -> lower=0 upper=3.14 effort=0.0 velocity=0.5; type revolute -> fixed
- joint right_hip: limit lower=-1.57 upper=1.57 effort=1000.0 velocity=0.5 -> lower=-1.57 upper=1.57 effort=0.0 velocity=0.5; origin xyz=0.000000 0.000000 0.339548 rpy=0 0 0 -> xyz=0.000000 0.000000 0.339548 rpy=0 0 0.384
- joint right_knee: limit lower=-3.14 upper=0. effort=0 velocity=200 -> lower=-3.14 upper=0. effort=0.0 velocity=0.5; origin xyz=0.000000 -1.686184 0.000000 rpy=0 0 0 -> xyz=0.000000 -1.686184 0.000000 rpy=0 0 -0.4712
- joint right_shoulder: type spherical -> fixed
- joint root: origin xyz=0.000000 0.000000 0.000000 rpy=0 0 0 -> xyz=0.000000 0.000000 0.000000 rpy=0 0 -0.1222
